Commit message: greedy exploration with tf_prefixed tree

File: src/kobuki_setup/kobuki_description/urdf/kobuki.urdf.xacro (robot description, xacro)
@@ -11,5 +11,5 @@
   <!-- Kobuki -->
   <xacro:macro name="kobuki">
-    <link name="base_footprint"/>
+    <link name="/qbot0/base_footprint"/>
     <!--
        Base link is set at the bottom of the base mould.
@@ -23,8 +23,8 @@
     <joint name="base_joint" type="fixed">
       <origin xyz="0 0 0.0102" rpy="0 0 0" />
-      <parent link="base_footprint"/>
-      <child link="base_link" />
-    </joint>
-    <link name="base_link">
+      <parent link="/qbot0/base_footprint"/>
+      <child link="/qbot0/base_link" />
+    </joint>
+    <link name="/qbot0/base_link">
       <visual>
         <geometry>
@@ -57,5 +57,5 @@
     </link>
     <joint name="wheel_left_joint" type="continuous">
-      <parent link="base_link"/>
+      <parent link="/qbot0/base_link"/>
       <child link="wheel_left_link"/>
       <origin xyz="0.00 ${0.23/2} 0.0250" rpy="${-M_PI/2} 0 0"/>
@@ -84,5 +84,5 @@
     </link>
     <joint name="wheel_right_joint" type="continuous">
-      <parent link="base_link"/>
+      <parent link="/qbot0/base_link"/>
       <child link="wheel_right_link"/>
       <origin xyz="0.00 -${0.23/2} 0.0250" rpy="${-M_PI/2} 0 0"/>
@@ -111,5 +111,5 @@
     </link>
     <joint name="caster_front_joint" type="fixed">
-      <parent link="base_link"/>
+      <parent link="/qbot0/base_link"/>
       <child link="caster_front_link"/>
       <origin xyz="0.115 0.0 0.007" rpy="${-M_PI/2} 0 0"/>
@@ -131,5 +131,5 @@
     </link>
     <joint name="caster_back_joint" type="fixed">
-      <parent link="base_link"/>
+      <parent link="/qbot0/base_link"/>
       <child link="caster_back_link"/>
       <origin xyz="-0.135 0.0 0.009" rpy="${-M_PI/2} 0 0"/>
@@ -154,5 +154,5 @@
       <axis xyz="0 1 0"/>
       <origin xyz="0.056 0.062 0.0202" rpy="0 0 0"/>
-      <parent link="base_link"/>
+      <parent link="/qbot0/base_link"/>
       <child link="gyro_link"/>
     </joint>
@@ -168,5 +168,5 @@
     <joint name="cliff_sensor_left_joint" type="fixed">
       <origin xyz="0.08734 0.13601 0.0214" rpy="0 ${M_PI/2} 0" />
-      <parent link="base_link"/>
+      <parent link="/qbot0/base_link"/>
       <child link="cliff_sensor_left_link" />
     </joint>
@@ -182,5 +182,5 @@
     <joint name="cliff_sensor_right_joint" type="fixed">
       <origin xyz="0.085 -0.13601 0.0214" rpy="0 ${M_PI/2} 0" />
-      <parent link="base_link"/>
+      <parent link="/qbot0/base_link"/>
       <child link="cliff_sensor_right_link" />
     </joint>
@@ -196,5 +196,5 @@
     <joint name="cliff_sensor_front_joint" type="fixed">
       <origin xyz="0.156 0.00 0.0214" rpy="0 ${M_PI/2} 0" />
-      <parent link="base_link"/>
+      <parent link="/qbot0/base_link"/>
       <child link="cliff_sensor_front_link" />
     </joint>
